File: board/board.kicad_pcb (KiCad board)
At the start: 2 copper layers, 21 x 13 mm, 1 part

Commit message: placed and routed
Parts:
- added C1: 100nF, Capacitor_SMD:C_0603_1608Metric, B.Cu at (155.7, 107.3)
- added C2: 100nF, Capacitor_SMD:C_0603_1608Metric, B.Cu at (155.7, 103.5)
- added C3: 100nF, Capacitor_SMD:C_0402_1005Metric, F.Cu at (145.6, 109.3)
- added C4: 100nF, Capacitor_SMD:C_0603_1608Metric, F.Cu at (155.9, 108.8)
- added C5: 100nF, Capacitor_SMD:C_0603_1608Metric, B.Cu at (155.7, 95.9)
- added C6: 100nF, Capacitor_SMD:C_0603_1608Metric, B.Cu at (155.6, 99.7)
- added D1: SMBJ58A-FDICT-ND, Diode_SMD:D_SMB, F.Cu at (153.5, 105.8)
- added D2: SMBJ58A-FDICT-ND, Diode_SMD:D_SMB, F.Cu at (153.5, 101.3)
- added D3: SMBJ58A-FDICT-ND, Diode_SMD:D_SMB, F.Cu at (153.5, 92.3)
- added D4: SMBJ58A-FDICT-ND, Diode_SMD:D_SMB, F.Cu at (153.5, 96.8)
- added F1: 60VDC, Fuse:Fuse_1206_3216Metric, B.Cu at (154.9, 105.4)
- added F2: 60VDC, Fuse:Fuse_1206_3216Metric, B.Cu at (154.9, 101.6)
- added F3: 60VDC, Fuse:Fuse_1206_3216Metric, B.Cu at (154.9, 94.0)
- added F4: 60VDC, Fuse:Fuse_1206_3216Metric, B.Cu at (154.8, 97.8)
- added J1: 001_I2C, on_edge:on_edge_2x05_device, F.Cu at (140.0, 97.0)
- added J2: Conn_01x06_Male, Connector_PinHeader_2.54mm:PinHeader_1x06_P2.54mm_Vertical, F.Cu at (159.0, 93.0)
- added Q1: SSM3K361R, Package_TO_SOT_SMD:SOT-23, B.Cu at (143.4, 116.9)
- added Q2: SSM3K361R, Package_TO_SOT_SMD:SOT-23, B.Cu at (143.4, 113.0)
- added Q3: SSM3K361R, Package_TO_SOT_SMD:SOT-23, B.Cu at (157.7, 112.8)
- added Q4: SSM3K361R, Package_TO_SOT_SMD:SOT-23, B.Cu at (157.6, 116.7)
- added R1: 0.51R, Resistor_SMD:R_0603_1608Metric, F.Cu at (142.8, 116.8)
- added R10: 47R, Resistor_SMD:R_0603_1608Metric, F.Cu at (155.9, 116.6)
- added R11: 22.1R, Resistor_SMD:R_0603_1608Metric, F.Cu at (155.9, 118.1)
- added R12: 22.1R, Resistor_SMD:R_0603_1608Metric, F.Cu at (155.9, 115.1)
- added R13: 0.51R, Resistor_SMD:R_0603_1608Metric, F.Cu at (158.2, 114.0)
- added R14: 0.51R, Resistor_SMD:R_0603_1608Metric, F.Cu at (158.2, 116.9)
- added R15: 0.51R, Resistor_SMD:R_0603_1608Metric, F.Cu at (159.7, 114.0)
- added R16: 0.51R, Resistor_SMD:R_0603_1608Metric, F.Cu at (159.7, 116.9)
- added R2: 0.51R, Resistor_SMD:R_0603_1608Metric, F.Cu at (141.3, 116.8)
- added R3: 47R, Resistor_SMD:R_0603_1608Metric, F.Cu at (145.1, 117.9)
- added R4: 22.1R, Resistor_SMD:R_0603_1608Metric, F.Cu at (145.1, 116.4)
- added R5: 0.51R, Resistor_SMD:R_0603_1608Metric, F.Cu at (141.3, 113.9)
- added R6: 0.51R, Resistor_SMD:R_0603_1608Metric, F.Cu at (142.8, 113.9)
- added R7: 47R, Resistor_SMD:R_0603_1608Metric, F.Cu at (145.1, 114.7)
- added R8: 22.1R, Resistor_SMD:R_0603_1608Metric, F.Cu at (145.1, 113.2)
- added R9: 47R, Resistor_SMD:R_0603_1608Metric, F.Cu at (155.9, 113.6)
- added U1: TPS23861, Package_SO:TSSOP-28_4.4x9.7mm_P0.65mm, F.Cu at (150.5, 113.5)
- moved LOGO1 8.99 mm to (143.4, 105.1)
Routing:
- net GND: track 0.00 -> 101.5 mm, vias 0 -> 7
- net /poe_pse/PoE+: track 0.00 -> 42.5 mm, vias 0 -> 2
- net /poe_pse/SW1: track 0.00 -> 33.4 mm, vias 0 -> 3
- net /poe_pse/SW2: track 0.00 -> 26.4 mm, vias 0 -> 3
- net /poe_pse/SDAI: track 0.00 -> 25.9 mm, vias 0 -> 2
- net +3.3V: track 0.00 -> 23.2 mm, vias 0 -> 1
- net /poe_pse/SCL: track 0.00 -> 22.1 mm
- net /poe_pse/SW4: track 0.00 -> 21.8 mm, vias 0 -> 1
- net /poe_pse/SW3: track 0.00 -> 21.1 mm, vias 0 -> 1
- net /poe_pse/INT: track 0.00 -> 19.6 mm
- net /poe_pse/switch2: track 0.00 -> 10.3 mm
- net /poe_pse/gate1: track 0.00 -> 8.91 mm, vias 0 -> 1
- net /poe_pse/switch3: track 0.00 -> 8.86 mm
- net /poe_pse/switch1: track 0.00 -> 8.77 mm, vias 0 -> 1
- net /poe_pse/switch4: track 0.00 -> 8.18 mm
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Other:
- board size 21 x 13 mm -> 21 x 29 mm
- board text added: "osf.001"
- board text added: "osf.b115.v1.0"
